File: defcon_key.kicad_pcb (KiCad board)
At the start: 2 copper layers, 83.8 x 119.4 mm, 22 parts, among them U1 ATTINY84-20PU

Commit message: Huge amount of code worked on. Need to push badge design upgrades.
Parts:
- moved BTTN1 49.7 mm to (95.2, 94.0)
- moved U1 17.0 mm to (91.4, 61.0), turned to 270 degrees
- moved R9 16.5 mm to (86.4, 73.7), turned to 90 degrees
- moved R1 2.54 mm to (83.8, 88.9)
- moved R2 2.54 mm to (83.8, 97.8)
- moved R3 2.54 mm to (83.8, 106.7)
- moved R4 2.54 mm to (83.8, 115.6)
- moved R5 2.54 mm to (83.8, 124.5)
- moved R6 2.54 mm to (83.8, 133.3)
- moved R7 2.54 mm to (83.8, 142.2)
- moved R8 2.54 mm to (83.8, 151.1)
Routing:
- net Net-(R8-Pad2): track 0.00 -> 152.5 mm
- net Net-(BT1-Pad2): track 0.00 -> 108.2 mm
- net Net-(R7-Pad2): track 0.00 -> 93.3 mm
- net Net-(R6-Pad2): track 0.00 -> 82.3 mm
- net Net-(R5-Pad2): track 0.00 -> 62.2 mm
- net Net-(R4-Pad2): track 0.00 -> 57.9 mm
- net Net-(BT1-Pad1): track 0.00 -> 55.8 mm
- net Net-(R3-Pad2): track 0.00 -> 48.3 mm
- net Net-(EYELED1-Pad2): track 0.00 -> 47.9 mm
- net Net-(R2-Pad2): track 0.00 -> 41.7 mm
- net Net-(R1-Pad2): track 0.00 -> 38.6 mm
- net Net-(BTTN1-Pad2): track 0.00 -> 26.9 mm
- net Net-(R9-Pad2): track 0.00 -> 12.3 mm
- net Net-(LED8-Pad2): track 0.00 -> 3.81 mm
- net Net-(LED7-Pad2): track 0.00 -> 3.81 mm
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Other:
- board text added: "The Shogun of Sorrow"

Commit message: Updates!
Parts:
- added RDOWN1: R, Resistors_THT:R_Axial_DIN0207_L6.3mm_D2.5mm_P7.62mm_Horizontal, B.Cu at (91.4, 77.5)
- BTTN1: footprint Buttons_Switches_THT:SW_PUSH-12mm -> Buttons_Switches_THT:SW_PUSH_6mm
- LED1, LED2, LED3, LED4, LED5, LED6, LED7, LED8: footprint LEDs:LED_D5.0mm -> LEDs:LED_D3.0mm
- moved LED1 17.8 mm to (77.5, 106.7)
- moved LED3 17.8 mm to (77.5, 88.9)
- moved R1 17.8 mm to (83.8, 106.7)
- moved R3 17.8 mm to (83.8, 88.9)
- moved U1 17.0 mm to (106.7, 68.6), turned to 90 degrees
- moved BTTN1 9.92 mm to (101.6, 86.4)
Connections:
- U1 pad 11: Net-(R2-Pad2) -> Net-(BTTN1-Pad2)
- U1 pad 12: Net-(R1-Pad2) -> Net-(R2-Pad2)
- U1 pad 13: Net-(BTTN1-Pad2) -> Net-(R1-Pad2)
- U1 pad 2: Net-(R8-Pad2) -> Net-(U1-Pad2)
- U1 pad 3: Net-(R9-Pad2) -> Net-(R8-Pad2)
- U1 pad 5: Net-(U1-Pad5) -> Net-(R7-Pad2)
- U1 pad 6: Net-(R7-Pad2) -> Net-(R6-Pad2)
- U1 pad 7: Net-(R6-Pad2) -> Net-(R5-Pad2)
- U1 pad 8: Net-(R5-Pad2) -> Net-(R9-Pad2)
Routing:
- net Net-(BT1-Pad2): track 108.2 -> 187.2 mm
- net Net-(R8-Pad2): track 152.5 -> 104.7 mm
- net Net-(BT1-Pad1): track 55.8 -> 100.0 mm
- net Net-(R5-Pad2): track 62.2 -> 89.3 mm
- net Net-(R4-Pad2): track 57.9 -> 81.9 mm
- net Net-(EYELED1-Pad2): track 47.9 -> 25.7 mm
- net Net-(R1-Pad2): track 38.6 -> 55.9 mm
- net Net-(BTTN1-Pad2): track 26.9 -> 39.6 mm
- net Net-(R7-Pad2): track 93.3 -> 102.7 mm
- net Net-(R2-Pad2): track 41.7 -> 47.8 mm
- net Net-(R3-Pad2): track 48.3 -> 44.4 mm
- net Net-(R9-Pad2): track 12.3 -> 8.67 mm
- net Net-(R6-Pad2): track 82.3 -> 83.8 mm
