File: defcon_key.sch (KiCad schematic (older format))
At the start: 12 parts, among them U1 ATTINY84-20PU

Commit message: IMPROVEMENTS!
Parts:
- added EYELED2: LED, LEDs:LED_D5.0mm, symbol LED
- added R1, R2, R3, R4, R5, R6, R7, R8, R9: R, Resistors_THT:R_Axial_DIN0207_L6.3mm_D2.5mm_P7.62mm_Horizontal, symbol R
- BT1: footprint (none) -> Battery_Holders:Keystone_103_1x20mm-CoinCell
- BTTN1: footprint (none) -> Buttons_Switches_THT:SW_PUSH-12mm
- EYELED1: renamed from LED9; footprint (none) -> LEDs:LED_D5.0mm
- LED1, LED2, LED3, LED4, LED5, LED6, LED7, LED8: footprint (none) -> LEDs:LED_D5.0mm
Connections:
- net at U1.10 ((PCINT3/T0/ADC3)PA3): now also R3.2
- net at U1.11 ((PCINT2/AIN1/ADC2)PA2): now also R2.2
- net at U1.12 ((PCINT1/AIN0/ADC1)PA1): now also R1.2
- net at BT1.2 (-), U1.14 (GND): now also EYELED1.1 (K), LED1.1 (K), LED2.1 (K), LED3.1 (K), LED4.1 (K), LED5.1 (K), LED6.1 (K), LED7.1 (K), LED8.1 (K), EYELED2.1 (K)
- net at U1.2 ((PCINT8/CLKI/XTAL1)PB0): now also R8.2
- net at U1.3 ((PCINT9/XTAL2)PB1): now also R9.2
- net at U1.6 ((PCINT7/ICP/OC0B/ADC7)PA7): now also R7.2
- net at U1.7 ((PCINT6/SDA/DI/MOSI/OC1A/ADC6)PA6): now also R6.2
- net at U1.8 ((PCINT5/DO/MISO/OC1B/ADC5)PA5): now also R5.2
- net at U1.9 ((PCINT4/USCK/SCL/T1/ADC4)PA4): now also R4.2
- net at LED2.2 (A): now also R2.1
- net at LED3.2 (A): now also R3.1
- net at LED4.2 (A): now also R4.1
- net at LED5.2 (A): now also R5.1
- net at LED6.2 (A): now also R6.1
- net at LED7.2 (A): now also R7.1
- net at LED1.2 (A): now also R1.1
- net at LED8.2 (A): now also R8.1
- net at EYELED1.2 (A): now also EYELED2.2 (A), R9.1
Other:
- moved on the sheet: EYELED1, LED1, LED2, LED3, LED4, LED5, LED6, LED7, LED8

Commit message: Updates!
Parts:
- added RDOWN1: R, Resistors_THT:R_Axial_DIN0207_L6.3mm_D2.5mm_P7.62mm_Horizontal, symbol R
- BTTN1: footprint Buttons_Switches_THT:SW_PUSH-12mm -> Buttons_Switches_THT:SW_PUSH_6mm
- LED1, LED2, LED3, LED4, LED5, LED6, LED7, LED8: footprint LEDs:LED_D5.0mm -> LEDs:LED_D3.0mm
Connections:
- net at U1.11 ((PCINT2/AIN1/ADC2)PA2): now also BTTN1.2 (B), RDOWN1.2; no longer R2.2
- net at U1.12 ((PCINT1/AIN0/ADC1)PA1): now also R2.2; no longer R1.2
- net at U1.13 ((PCINT0/AREF/ADC0)PA0): now also R1.2; no longer BTTN1.2 (B)
- net at BT1.2 (-), EYELED1.1 (K), EYELED2.1 (K)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: now also RDOWN1.1
- net at U1.2 ((PCINT8/CLKI/XTAL1)PB0): no longer R8.2
- net at U1.3 ((PCINT9/XTAL2)PB1): now also R8.2; no longer R9.2
- net at U1.5 ((PCINT10/CKOUT/OC0A/INT0)PB2): now also R7.2
- net at U1.6 ((PCINT7/ICP/OC0B/ADC7)PA7): now also R6.2; no longer R7.2
- net at U1.7 ((PCINT6/SDA/DI/MOSI/OC1A/ADC6)PA6): now also R5.2; no longer R6.2
- net at U1.8 ((PCINT5/DO/MISO/OC1B/ADC5)PA5): now also R9.2; no longer R5.2
Other:
- moved on the sheet: BTTN1, LED1, LED2, R1, R2
Changed lines of the file:
@@
 L SW_Push_Open BTTN1
 U 1 1 5AE00593
-P 3350 3450
-F 0 "BTTN1" H 3350 3550 50  0000 C CNN
-F 1 "Push Button" H 3350 3375 50  0000 C CNN
-F 2 "Buttons_Switches_THT:SW_PUSH-12mm" H 3350 3650 50  0001 C CNN
-F 3 "" H 3350 3650 50  0001 C CNN
-	1    3350 3450
+P 5000 2950
+F 0 "BTTN1" H 5000 3050 50  0000 C CNN
+F 1 "Push Button" H 5000 2875 50  0000 C CNN
+F 2 "Buttons_Switches_THT:SW_PUSH_6mm" H 5000 3150 50  0001 C CNN
+F 3 "" H 5000 3150 50  0001 C CNN
+	1    5000 2950
 	1    0    0    -1
 $EndComp
@@
 L LED LED2
 U 1 1 5AE006C5
-P 5500 3800
-F 0 "LED2" H 5500 3900 50  0000 C CNN
-F 1 "LED" H 5500 3700 50  0000 C CNN
-F 2 "LEDs:LED_D5.0mm" H 5500 3800 50  0001 C CNN
-F 3 "" H 5500 3800 50  0001 C CNN
-	1    5500 3800
+P 5500 3600
+F 0 "LED2" H 5500 3700 50  0000 C CNN
+F 1 "LED" H 5500 3500 50  0000 C CNN
+F 2 "LEDs:LED_D3.0mm" H 5500 3600 50  0001 C CNN
+F 3 "" H 5500 3600 50  0001 C CNN
+	1    5500 3600
 	-1   0    0    -1
 $EndComp
@@
 F 0 "LED3" H 5500 4200 50  0000 C CNN
 F 1 "LED" H 5500 4000 50  0000 C CNN
-F 2 "LEDs:LED_D5.0mm" H 5500 4100 50  0001 C CNN
+F 2 "LEDs:LED_D3.0mm" H 5500 4100 50  0001 C CNN
 F 3 "" H 5500 4100 50  0001 C CNN
 	1    5500 4100
@@
 F 0 "LED4" H 5500 4500 50  0000 C CNN
 F 1 "LED" H 5500 4300 50  0000 C CNN
-F 2 "LEDs:LED_D5.0mm" H 5500 4400 50  0001 C CNN
+F 2 "LEDs:LED_D3.0mm" H 5500 4400 50  0001 C CNN
 F 3 "" H 5500 4400 50  0001 C CNN
 	1    5500 4400
@@
 F 0 "LED5" H 5500 4800 50  0000 C CNN
 F 1 "LED" H 5500 4600 50  0000 C CNN
-F 2 "LEDs:LED_D5.0mm" H 5500 4700 50  0001 C CNN
+F 2 "LEDs:LED_D3.0mm" H 5500 4700 50  0001 C CNN
 F 3 "" H 5500 4700 50  0001 C CNN
 	1    5500 4700
@@
 F 0 "LED6" H 5500 5100 50  0000 C CNN
 F 1 "LED" H 5500 4900 50  0000 C CNN
-F 2 "LEDs:LED_D5.0mm" H 5500 5000 50  0001 C CNN
+F 2 "LEDs:LED_D3.0mm" H 5500 5000 50  0001 C CNN
 F 3 "" H 5500 5000 50  0001 C CNN
 	1    5500 5000
@@
 F 0 "LED7" H 5500 5400 50  0000 C CNN
 F 1 "LED" H 5500 5200 50  0000 C CNN
-F 2 "LEDs:LED_D5.0mm" H 5500 5300 50  0001 C CNN
+F 2 "LEDs:LED_D3.0mm" H 5500 5300 50  0001 C CNN
 F 3 "" H 5500 5300 50  0001 C CNN
 	1    5500 5300
@@
 L LED LED1
 U 1 1 5AE00A21
-P 5500 3500
-F 0 "LED1" H 5500 3600 50  0000 C CNN
-F 1 "LED" H 5500 3400 50  0000 C CNN
-F 2 "LEDs:LED_D5.0mm" H 5500 3500 50  0001 C CNN
-F 3 "" H 5500 3500 50  0001 C CNN
-	1    5500 3500
+P 5500 3300
+F 0 "LED1" H 5500 3400 50  0000 C CNN
+F 1 "LED" H 5500 3200 50  0000 C CNN
+F 2 "LEDs:LED_D3.0mm" H 5500 3300 50  0001 C CNN
+F 3 "" H 5500 3300 50  0001 C CNN
+	1    5500 3300
 	-1   0    0    -1
 $EndComp
@@
 F 0 "LED8" H 5500 5700 50  0000 C CNN
 F 1 "LED" H 5500 5500 50  0000 C CNN
-F 2 "LEDs:LED_D5.0mm" H 5500 5600 50  0001 C CNN
+F 2 "LEDs:LED_D3.0mm" H 5500 5600 50  0001 C CNN
 F 3 "" H 5500 5600 50  0001 C CNN
 	1    5500 5600
@@
 	-1   0    0    -1
 $EndComp
-NoConn ~ 4350 4900
-NoConn ~ 4350 5000
 $Comp
 L Battery_Cell BT1
@@
 Wire Wire Line
 	1850 3450 1850 4250
-Wire Wire Line
-	4350 3450 4350 3800
-Wire Wire Line
-	3550 3450 4350 3450
 Connection ~ 2050 5000
 Wire Wire Line
@@
 	2050 4800 2050 6350
 Wire Wire Line
-	5150 3500 5350 3500
-Wire Wire Line
-	6050 3500 6050 6350
+	6050 2950 6050 6350
 Connection ~ 6050 5900
 Connection ~ 6050 5600
@@
 Connection ~ 6050 4400
 Connection ~ 6050 4100
-Connection ~ 6050 3800
-Wire Wire Line
-	4350 3900 4500 3900
-Wire Wire Line
-	4500 3900 4500 3500
-Wire Wire Line
-	4350 4700 4450 4700
-Wire Wire Line
-	4450 4700 4450 5600
-Wire Wire Line
-	4350 4500 4500 4500
-Wire Wire Line
-	4500 4500 4500 5300
 Wire Wire Line
 	5150 5300 5350 5300
@@
 L R R1
 U 1 1 5B123A70
-P 5000 3500
-F 0 "R1" V 5080 3500 50  0000 C CNN
-F 1 "R" V 5000 3500 50  0000 C CNN
-F 2 "Resistors_THT:R_Axial_DIN0207_L6.3mm_D2.5mm_P7.62mm_Horizontal" V 4930 3500 50  0001 C CNN
-F 3 "" H 5000 3500 50  0001 C CNN
-	1    5000 3500
+P 5000 3300
+F 0 "R1" V 5080 3300 50  0000 C CNN
+F 1 "R" V 5000 3300 50  0000 C CNN
+F 2 "Resistors_THT:R_Axial_DIN0207_L6.3mm_D2.5mm_P7.62mm_Horizontal" V 4930 3300 50  0001 C CNN
+F 3 "" H 5000 3300 50  0001 C CNN
+	1    5000 3300
 	0    1    1    0
 $EndComp
@@
 L R R2
 U 1 1 5B123B2E
-P 5000 3800
-F 0 "R2" V 5080 3800 50  0000 C CNN
-F 1 "R" V 5000 3800 50  0000 C CNN
-F 2 "Resistors_THT:R_Axial_DIN0207_L6.3mm_D2.5mm_P7.62mm_Horizontal" V 4930 3800 50  0001 C CNN
-F 3 "" H 5000 3800 50  0001 C CNN
-	1    5000 3800
+P 5000 3600
+F 0 "R2" V 5080 3600 50  0000 C CNN
+F 1 "R" V 5000 3600 50  0000 C CNN
+F 2 "Resistors_THT:R_Axial_DIN0207_L6.3mm_D2.5mm_P7.62mm_Horizontal" V 4930 3600 50  0001 C CNN
+F 3 "" H 5000 3600 50  0001 C CNN
+	1    5000 3600
 	0    1    1    0
 $EndComp
@@
 	5650 5900 6050 5900
 Wire Wire Line
-	4450 5600 4850 5600
-Wire Wire Line
 	5150 5600 5350 5600
 Wire Wire Line
@@
 	6050 5300 5650 5300
 Wire Wire Line
-	4500 5300 4850 5300
-Wire Wire Line
-	5150 3800 5350 3800
-Wire Wire Line
 	5150 4300 5350 4300
 Wire Wire Line
@@
 	5650 4100 6050 4100
 Wire Wire Line
-	6050 3500 5650 3500
-Wire Wire Line
-	5650 3800 6050 3800
-Wire Wire Line
-	4500 3500 4850 3500
-Wire Wire Line
-	4850 3800 4650 3800
-Wire Wire Line
-	4650 3800 4650 4000
-Wire Wire Line
-	4650 4000 4350 4000
-Wire Wire Line
 	4350 4100 4850 4100
 Wire Wire Line
@@
 	4850 4200 4850 4300
 Wire Wire Line
-	4350 4300 4800 4300
-Wire Wire Line
-	4800 4300 4800 4700
-Wire Wire Line
 	4800 4700 4850 4700
-Wire Wire Line
-	4350 4400 4650 4400
-Wire Wire Line
-	4650 4400 4650 5000
-Wire Wire Line
-	4650 5000 4850 5000
-Wire Wire Line
-	4350 4800 4400 4800
-Wire Wire Line
-	4400 4800 4400 5900
-Wire Wire Line
-	4400 5900 4850 5900
 Wire Wire Line
 	5150 4100 5350 4100
@@
 	5650 6200 6050 6200
 Connection ~ 6050 6200
+$Comp
+L R RDOWN1
+U 1 1 5B44FDBE
+P 5500 2950
+F 0 "RDOWN1" V 5580 2950 50  0000 C CNN
+F 1 "R" V 5500 2950 50  0000 C CNN
+F 2 "Resistors_THT:R_Axial_DIN0207_L6.3mm_D2.5mm_P7.62mm_Horizontal" V 5430 2950 50  0001 C CNN
+F 3 "" H 5500 2950 50  0001 C CNN
+	1    5500 2950
+	0    1    1    0
+$EndComp
+Wire Wire Line
+	4350 3800 4350 3300
+Wire Wire Line
+	4350 3300 4850 3300
+Wire Wire Line
+	5150 3300 5350 3300
+Wire Wire Line
+	4350 3900 4450 3900
+Wire Wire Line
+	4450 3900 4450 3600
+Wire Wire Line
+	4450 3600 4850 3600
+Wire Wire Line
+	5150 3600 5350 3600
+Wire Wire Line
+	4350 4000 5250 4000
+Wire Wire Line
+	5200 2950 5350 2950
+Connection ~ 5250 2950
+Wire Wire Line
+	5250 4000 5250 2950
+Wire Wire Line
+	4800 2950 3150 2950
+Wire Wire Line
+	3150 2950 3150 3450
+Wire Wire Line
+	5650 2950 6050 2950
+Wire Wire Line
+	5650 3300 6050 3300
+Connection ~ 6050 3300
+Wire Wire Line
+	5650 3600 6050 3600
+Connection ~ 6050 3600
+Wire Wire Line
+	4350 4300 4550 4300
+Wire Wire Line
+	4550 4300 4550 5900
+Wire Wire Line
+	4550 5900 4850 5900
+Wire Wire Line
+	4350 4400 4800 4400
+Wire Wire Line
+	4800 4400 4800 4700
+Wire Wire Line
+	4350 4500 4700 4500
+Wire Wire Line
+	4700 4500 4700 5000
+Wire Wire Line
+	4700 5000 4850 5000
+Wire Wire Line
+	4350 4900 4650 4900
+Wire Wire Line
+	4650 4900 4650 5300
+Wire Wire Line
+	4650 5300 4850 5300
+Wire Wire Line
+	4350 4800 4600 4800
+Wire Wire Line
+	4600 4800 4600 5600
+Wire Wire Line
+	4600 5600 4850 5600
+NoConn ~ 4350 4700
+NoConn ~ 4350 5000
 $EndSCHEMATC
